File: ZeroCrossDetector.kicad_pcb (KiCad board)
At the start: 2 copper layers, 85 x 85 mm, 72 parts, among them J1 POWER, J2 BCKUP_CON, J3 BNC, J4 BNC, J5 BCKUP_CON, J6 BNC, J7 BNC, U1 AD8041, U2 AD8041, U3 RKJXL100401V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

Commit message: resistor values decreased
Parts:
- R10: value 47M 1% -> 10M 1%
- R11: value 10M 1% -> 2M2 1%
- R12: value 4M7 1% -> 1M 1%
- R13: value 1M 1% -> 220k 1%
- R14: value 470k 1% -> 100k 1%
- R15: value 100k 1% -> 20k 1%
- R16: value 47k 1% -> 10k 1%
- R18: value 100M 1% -> 22M 1%
- R7: value 4k7 1% -> 1k 1%
- R8: value 1Meg 1% -> 220k 1%
- turned R13 to 0 degrees
Connections:
- D5 pad 1: GND -> unconnected-(D5-Pad1)
- R13 pad 1: Net-(C16-Pad1) -> Net-(U3-PadE)
- R13 pad 2: Net-(R13-Pad2) -> Net-(C16-Pad1)
- U3 pad E: Net-(R13-Pad2) -> Net-(U3-PadE)
Routing:
- net Net-(U3-PadE): track 0.00 -> 9.89 mm
- net Net-(R13-Pad2): track 9.89 -> 0.00 mm
- net GND: track 410.4 -> 408.3 mm
