File: ZeroCrossDetector.kicad_sch (KiCad schematic)
At the start: 68 parts, among them J1 POWER, J2 BCKUP_CON, J3 BNC, J4 BNC, J5 BCKUP_CON, J6 BNC, J7 BNC, U1 AD8041, U2 AD8041, U3 RKJXL100401V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

Commit message: resistor values decreased
Parts:
- R10: value 47M 1% -> 10M 1%; JLC C137426 -> C26108
- R11: value 10M 1% -> 2M2 1%; JLC C26108 -> C26113
- R12: value 4M7 1% -> 1M 1%; JLC C413240 -> C17514
- R13: value 1M 1% -> 220k 1%; JLC C17514 -> C17556
- R14: value 470k 1% -> 100k 1%; JLC C17709 -> C149504
- R15: value 100k 1% -> 20k 1%; JLC C149504 -> C4328
- R16: value 47k 1% -> 10k 1%; JLC C17713 -> C17414
- R18: value 100M 1% -> 22M 1%; JLC C137480 -> C62398
- R7: value 4k7 1% -> 1k 1%; JLC C17673 -> C17513
- R8: value 1Meg 1% -> 220k 1%; JLC C17514 -> C17556
Connections:
- net GND: no longer D5.1
- net at U3.E: now also R13.1; no longer R13.2
- net at C16.1, R10.1, R11.1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: now also R13.2; no longer R13.1
- no-connect marks 0 -> 1
